File: joyMIDI/joyMIDI.kicad_pcb (KiCad board)
At the start: 2 copper layers, 140 x 76.9 mm, 222 parts, among them J1 USB_C_Receptacle/Amphenol_124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, J2 HDR_01X04, J3 SJ-2524-SMT, J4 HDR_01X04, J5 HDR_01X05, SW1 SW, SW10 SW, SW11 SW, SW12 SW, SW13 SW, SW14 SW, SW15 SW, SW16 SW, SW17 SW, SW18 SW, SW19 SW, SW2 SW, SW20 SW, SW3 SW, SW4 SW, SW5 SW, SW6 SW, SW7 SW, SW8 SW, SW9 SW, U1 AIC1746-33, U10 74HC165, U2 M452LD3AE, U3 BMA2xx, U4 74HC595, U5 74HC165, U6 74HC595, U7 74HC165, U8 TLP2361, U9 74HC595, Y1 12M

Commit message: V1.0 2019.5 Change USB connector to 16pin from 24pin Add placement file for SMT
Parts:
- C10, C6: value 4.7u/0805 -> 4.7u
- J1: value USB_C_Receptacle/Amphenol_12401610E4#2A -> USB_Type_C_16P; footprint Connector_USB:USB_C_Receptacle_Amphenol_12401610E4-2A -> joyMIDI:HRO_TYPE-C-31-M-12
- J3: value SJ-2524-SMT -> AUDIO_JACK_TRS_4P_2.5mm
- R33: value 2K -> 3.3K
- U2: value M452LD3AE -> M452LE6AE
- moved J1 5.11 mm to (176.0, 64.6)
- moved G*** 3.15 mm to (90.0, 73.0)
Connections:
- J1 pad A8: Net-(J1-PadA8) -> (no net)
- J1 pad B8: Net-(J1-PadB8) -> (no net)
- J3 pad 1: Net-(J3-Pad1) -> (no net)
- J3 pad 4: Net-(J3-Pad4) -> (no net)
- L1 pad 2: Net-(J1-PadS1) -> Net-(J1-PadSH)
- U10 pad 7: Net-(U10-Pad7) -> (no net)
- U2 pad 11: Net-(U2-Pad11) -> (no net)
- U2 pad 12: Net-(U2-Pad12) -> (no net)
- U2 pad 13: Net-(U2-Pad13) -> (no net)
- U2 pad 14: Net-(U2-Pad14) -> (no net)
- U2 pad 19: Net-(U2-Pad19) -> (no net)
- U2 pad 3: Net-(U2-Pad3) -> (no net)
- U2 pad 30: Net-(U2-Pad30) -> (no net)
- U2 pad 35: Net-(U2-Pad35) -> (no net)
- U2 pad 44: Net-(U2-Pad44) -> (no net)
- U3 pad 10: Net-(U3-Pad10) -> (no net)
- U3 pad 5: Net-(U3-Pad5) -> (no net)
- U3 pad 6: Net-(U3-Pad6) -> (no net)
- U4 pad 4: Net-(U4-Pad4) -> (no net)
- U4 pad 5: Net-(U4-Pad5) -> (no net)
- U4 pad 6: Net-(U4-Pad6) -> (no net)
- U4 pad 7: Net-(U4-Pad7) -> (no net)
- U4 pad 9: Net-(U4-Pad9) -> (no net)
- U5 pad 10: Net-(U5-Pad10) -> (no net)
- U5 pad 7: Net-(U5-Pad7) -> (no net)
- U7 pad 7: Net-(U7-Pad7) -> (no net)
Routing:
- net Net-(J1-PadSH): track 0.00 -> 5.15 mm
- net Net-(J1-PadS1): track 3.78 -> 0.00 mm
- net VBUS: track 15.1 -> 18.3 mm, vias 2 -> 0
- net /D+: track 11.9 -> 14.7 mm, vias 2 -> 0
- net /D-: track 11.5 -> 13.5 mm, vias 2 -> 0
- net VCC_DIG: track 825.0 -> 826.5 mm
- net Net-(J1-PadA5): track 10.9 -> 11.5 mm
- net GND_PWR: track 37.4 -> 37.2 mm, vias 15 -> 17
Other:
- board text added: "joyMIDI V1.0_2019.5"
- board text removed: "joyMIDI V4.0_2019.2"
