File: joyMIDI/joyMIDI.kicad_pcb (KiCad board)
At the start: 2 copper layers, 140 x 76.9 mm, 222 parts, among them J1 USB_Type_C_16P, J2 HDR_01X04, J3 AUDIO_JACK_TRS_4P_2.5mm, J4 HDR_01X04, J5 HDR_01X05, SW1 SW, SW10 SW, SW11 SW, SW12 SW, SW13 SW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

Commit message: Change Logo
Parts:
- removed the G*** at (90.0, 73.0)
- added G***: LOGO, joyMIDI:Logo_Soundless_25x3p6, F.Cu at (112.1, 74.6)
Other:
- board text added: "joyMIDI V1.0_2019.8"
- board text removed: "joyMIDI V1.0_2019.5"
